File: tps5430.kicad_sch (KiCad schematic)
At the start: 12 parts, among them J1 Conn_01x01_Pin, J2 Conn_01x01_Pin, J3 Conn_01x01_Pin, J4 Conn_01x01_Pin

Commit message: final
Parts:
- U?: footprint Package_SO:TI_SO-PowerPAD-8_ThermalVias -> footprints:TI_SO-PowerPAD-8_ThermalVias
Changed lines of the file:
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@@
       (effects (font (size 1.27 1.27)))
     )
-    (property "Footprint" "Package_SO:TI_SO-PowerPAD-8_ThermalVias" (at 129.54 109.22 0)
+    (property "Footprint" "footprints:TI_SO-PowerPAD-8_ThermalVias" (at 129.54 109.22 0)
       (effects (font (size 1.27 1.27) italic) (justify left) hide)
     )
