File: tps5430.kicad_pcb (KiCad board)
At the start: 2 copper layers, 17.5 x 22 mm, 12 parts, among them J1 Conn_01x01_Pin, J2 Conn_01x01_Pin, J3 Conn_01x01_Pin, J4 Conn_01x01_Pin, U1 TPS5430DDA

Commit message: drc errors
Parts:
- U1: footprint Package_SO:TI_SO-PowerPAD-8_ThermalVias -> footprints:TI_SO-PowerPAD-8_ThermalVias
- moved C3 0.50 mm to (102.7, 46.4)
- moved C1 0.40 mm to (91.4, 44.5)
- moved R1 0.40 mm to (91.4, 46.4)
- moved R2 0.40 mm to (91.4, 48.3)
Routing:
- net GND: track 2.97 -> 0.00 mm
- net +5V: track 25.7 -> 24.4 mm

Commit message: final
Parts:
- moved C1 0.30 mm to (91.7, 44.5)
- moved C3 0.30 mm to (102.4, 46.4)
- moved R1 0.30 mm to (91.7, 46.4)
- moved R2 0.30 mm to (91.7, 48.3)
Routing:
- net +12V: track 8.39 -> 7.71 mm
- net Net-(D1-K): track 22.4 -> 21.9 mm
